File: hardware/ygl_energy_monitor.brd (EAGLE design)
At the start: 73.5 x 52 mm, 5 parts

Commit message: embrace the braze!
Parts:
- removed SV1: (no value), con-lstb:MA03-1
- added IC1: ACS750LCA-050, allegro:ACS75050
Connections:
- net N$1: now also IC1.1; no longer SV1.1
- net N$2: now also IC1.2; no longer SV1.2
- net N$3: now also IC1.3; no longer SV1.3
Routing:
- net N$2: track 18.8 -> 13.5 mm
- net N$1: track 23.3 -> 18.8 mm
- net N$3: track 48.4 -> 50.7 mm
Changed lines of the file:
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@@
 <hole x="62.992" y="10.7696" drill="3.175"/>
 <hole x="63.119" y="58.5216" drill="3.175"/>
-<rectangle x1="13.8684" y1="48.9204" x2="20.1168" y2="51.1556" layer="16"/>
-<rectangle x1="13.8938" y1="46.2788" x2="20.1422" y2="48.514" layer="16"/>
-<rectangle x1="13.8938" y1="43.688" x2="20.1422" y2="45.9232" layer="16"/>
-<rectangle x1="13.8938" y1="41.1988" x2="20.1422" y2="43.434" layer="16"/>
-<rectangle x1="13.8938" y1="38.6588" x2="20.1422" y2="40.894" layer="16"/>
-<rectangle x1="13.8938" y1="36.068" x2="20.1422" y2="38.3032" layer="16"/>
-<rectangle x1="13.8684" y1="33.5788" x2="20.1168" y2="35.814" layer="16"/>
-<rectangle x1="13.8684" y1="31.115" x2="20.1168" y2="33.3502" layer="16"/>
-<rectangle x1="13.8684" y1="28.4988" x2="20.1168" y2="30.734" layer="16"/>
-<rectangle x1="13.8938" y1="26.035" x2="20.1422" y2="28.2702" layer="16"/>
-<rectangle x1="13.8938" y1="23.495" x2="20.1422" y2="25.7302" layer="16"/>
-<rectangle x1="13.9446" y1="20.9804" x2="20.193" y2="23.2156" layer="16"/>
-<rectangle x1="30.4292" y1="48.9204" x2="36.6776" y2="51.1556" layer="16"/>
-<rectangle x1="30.4546" y1="46.2788" x2="36.703" y2="48.514" layer="16"/>
-<rectangle x1="30.4546" y1="43.688" x2="36.703" y2="45.9232" layer="16"/>
-<rectangle x1="30.4546" y1="41.1988" x2="36.703" y2="43.434" layer="16"/>
-<rectangle x1="30.4546" y1="38.6588" x2="36.703" y2="40.894" layer="16"/>
-<rectangle x1="30.4546" y1="36.068" x2="36.703" y2="38.3032" layer="16"/>
-<rectangle x1="30.4292" y1="33.5788" x2="36.6776" y2="35.814" layer="16"/>
-<rectangle x1="30.4292" y1="31.115" x2="36.6776" y2="33.3502" layer="16"/>
-<rectangle x1="30.4292" y1="28.4988" x2="36.6776" y2="30.734" layer="16"/>
-<rectangle x1="30.4546" y1="26.035" x2="36.703" y2="28.2702" layer="16"/>
-<rectangle x1="30.4546" y1="23.495" x2="36.703" y2="25.7302" layer="16"/>
-<rectangle x1="30.5054" y1="20.9804" x2="36.7538" y2="23.2156" layer="16"/>
 <rectangle x1="0.6096" y1="58.0898" x2="0.8382" y2="58.2168" layer="16"/>
-<rectangle x1="60.071" y1="38.608" x2="70.5612" y2="52.2224" layer="45"/>
-<rectangle x1="60.071" y1="16.5354" x2="70.5612" y2="30.1498" layer="45"/>
-<rectangle x1="50.6222" y1="36.8046" x2="73.2028" y2="56.2864" layer="16"/>
-<rectangle x1="50.6984" y1="12.9794" x2="73.279" y2="32.4612" layer="16"/>
+<rectangle x1="57.9882" y1="18.5928" x2="70.9676" y2="35.6362" layer="16"/>
+<rectangle x1="58.0644" y1="36.6014" x2="71.0438" y2="53.6448" layer="16"/>
+<rectangle x1="59.055" y1="36.6014" x2="65.5574" y2="49.276" layer="45"/>
+<rectangle x1="59.055" y1="22.987" x2="65.5574" y2="35.6616" layer="45"/>
 </plain>
 <attributes>
@@
 <element name="R2" library="resistor" library_urn="urn:adsk.eagle:library:348" package="0207/10" package3d_urn="urn:adsk.eagle:package:25939/1" value="" x="10.4902" y="19.6596" rot="R90"/>
 <element name="R1" library="resistor" library_urn="urn:adsk.eagle:library:348" package="0207/10" package3d_urn="urn:adsk.eagle:package:25939/1" value="" x="10.3378" y="33.1724" rot="R270"/>
-<element name="SV1" library="con-lstb" library_urn="urn:adsk.eagle:library:162" package="MA03-1" package3d_urn="urn:adsk.eagle:package:8339/1" value="" x="44.1706" y="34.2646" rot="R270">
-<attribute name="MF" value="" x="44.1706" y="34.2646" size="1.778" layer="27" rot="R270" display="off"/>
-<attribute name="MPN" value="" x="44.1706" y="34.2646" size="1.778" layer="27" rot="R270" display="off"/>
-<attribute name="OC_FARNELL" value="unknown" x="44.1706" y="34.2646" size="1.778" layer="27" rot="R270" display="off"/>
-<attribute name="OC_NEWARK" value="unknown" x="44.1706" y="34.2646" size="1.778" layer="27" rot="R270" display="off"/>
+<element name="IC1" library="allegro" library_urn="urn:adsk.eagle:library:93" package="ACS75050" package3d_urn="urn:adsk.eagle:package:3457/1" value="ACS750LCA-050" x="62.2554" y="36.068" rot="R270">
+<attribute name="MF" value="ALLEGRO MICROSYSTEMS, INC." x="62.2554" y="36.068" size="1.778" layer="27" rot="R270" display="off"/>
+<attribute name="MPN" value="ACS750LCA-050" x="62.2554" y="36.068" size="1.778" layer="27" rot="R270" display="off"/>
+<attribute name="OC_FARNELL" value="1457176" x="62.2554" y="36.068" size="1.778" layer="27" rot="R270" display="off"/>
+<attribute name="OC_NEWARK" value="61H4464" x="62.2554" y="36.068" size="1.778" layer="27" rot="R270" display="off"/>
 </element>
 </elements>
@@
 <contactref element="U$1" pad="24"/>
 <wire x1="34.29" y1="49.8856" x2="34.29" y2="50.038" width="0.6096" layer="16"/>
-<contactref element="SV1" pad="1"/>
-<wire x1="34.29" y1="50.038" x2="44.2214" y2="50.038" width="1.27" layer="16"/>
-<wire x1="44.2214" y1="50.038" x2="44.1706" y2="36.8046" width="1.27" layer="16"/>
+<contactref element="IC1" pad="1"/>
+<wire x1="34.29" y1="50.038" x2="40.8554" y2="50.038" width="1.5" layer="16"/>
+<wire x1="40.8554" y1="50.038" x2="40.8554" y2="37.978" width="1.5" layer="16"/>
 </signal>
 <signal name="N$2">
 <contactref element="U$1" pad="21"/>
 <wire x1="34.4678" y1="42.5196" x2="34.544" y2="41.91" width="0.4064" layer="16"/>
-<contactref element="SV1" pad="2"/>
-<wire x1="34.29" y1="42.418" x2="39.2176" y2="42.418" width="1.27" layer="16"/>
-<wire x1="39.1668" y1="34.2138" x2="44.1706" y2="34.2646" width="1.016" layer="16"/>
-<wire x1="39.2176" y1="42.418" x2="39.1668" y2="34.2138" width="1.27" layer="16"/>
+<contactref element="IC1" pad="2"/>
+<wire x1="40.8554" y1="36.068" x2="37.7444" y2="36.068" width="1.5" layer="16"/>
+<wire x1="37.7444" y1="36.068" x2="37.7444" y2="42.2656" width="1.5" layer="16"/>
+<wire x1="37.7444" y1="42.2656" x2="34.29" y2="42.2656" width="1.5" layer="16"/>
+<wire x1="34.29" y1="42.2656" x2="34.29" y2="42.418" width="1.27" layer="16"/>
 <wire x1="34.29" y1="42.418" x2="34.4678" y2="42.5196" width="0" layer="19" extent="16-16"/>
 </signal>
 <signal name="N$3">
 <contactref element="U$1" pad="12"/>
-<contactref element="SV1" pad="3"/>
-<wire x1="44.1706" y1="31.7246" x2="44.2214" y2="16.5862" width="1.27" layer="16"/>
-<wire x1="44.2214" y1="16.5862" x2="16.5608" y2="16.5862" width="1.27" layer="16"/>
-<wire x1="16.5608" y1="16.5862" x2="16.5608" y2="22.098" width="1.27" layer="16"/>
 <wire x1="16.5608" y1="22.098" x2="16.51" y2="22.098" width="0.508" layer="16"/>
+<contactref element="IC1" pad="3"/>
+<wire x1="16.51" y1="22.098" x2="16.51" y2="14.9606" width="1.5" layer="16"/>
+<wire x1="40.8554" y1="14.9606" x2="40.8554" y2="34.158" width="1.5" layer="16"/>
+<wire x1="16.51" y1="14.9606" x2="40.8554" y2="14.9606" width="1.5" layer="16"/>
 </signal>
 <signal name="VIN">
@@
 <contactref element="R1" pad="2"/>
 <wire x1="16.51" y1="24.6888" x2="16.51" y2="24.638" width="0.4064" layer="16"/>
-<wire x1="10.3378" y1="28.0924" x2="10.3378" y2="24.7396" width="1.27" layer="16"/>
+<wire x1="10.3378" y1="28.0924" x2="10.3378" y2="24.7396" width="1.5" layer="16"/>
 <wire x1="10.3378" y1="24.7396" x2="10.4902" y2="24.7396" width="0.6096" layer="16"/>
 <wire x1="10.4902" y1="24.7396" x2="10.4902" y2="24.6888" width="0.6096" layer="16"/>
-<wire x1="10.4902" y1="24.6888" x2="16.51" y2="24.6888" width="1.27" layer="16"/>
+<wire x1="10.4902" y1="24.6888" x2="16.51" y2="24.6888" width="1.5" layer="16"/>
 </signal>
 <signal name="N$4">
@@
 <contactref element="R1" pad="1"/>
 <contactref element="J2" pad="2"/>
-<wire x1="2.4638" y1="47.3404" x2="10.3378" y2="47.3404" width="1.27" layer="16"/>
-<wire x1="10.3378" y1="47.3404" x2="16.51" y2="47.3404" width="1.27" layer="16"/>
+<wire x1="2.4638" y1="47.3404" x2="10.3378" y2="47.3404" width="1.5" layer="16"/>
+<wire x1="10.3378" y1="47.3404" x2="16.51" y2="47.3404" width="1.5" layer="16"/>
 <wire x1="16.51" y1="47.3404" x2="16.51" y2="47.498" width="0.6096" layer="16"/>
-<wire x1="10.3378" y1="47.3404" x2="10.3378" y2="38.2524" width="1.27" layer="16"/>
+<wire x1="10.3378" y1="47.3404" x2="10.3378" y2="38.2524" width="1.5" layer="16"/>
 </signal>
 <signal name="N$5">
 <contactref element="J2" pad="1"/>
 <contactref element="R2" pad="1"/>
-<wire x1="2.4638" y1="43.8404" x2="2.4638" y2="14.5796" width="1.27" layer="16"/>
-<wire x1="2.4638" y1="14.5796" x2="10.4902" y2="14.5796" width="1.27" layer="16"/>
+<wire x1="2.4638" y1="43.8404" x2="2.4638" y2="14.5796" width="1.5" layer="16"/>
+<wire x1="2.4638" y1="14.5796" x2="10.4902" y2="14.5796" width="1.5" layer="16"/>
 </signal>
 </signals>

Commit message: fuck braze!
Parts:
- moved J2 3.33 mm to (5.79, 43.7)
Routing:
- net N$5: track 37.3 -> 33.9 mm
- net N$4: track 23.3 -> 20.0 mm
Other:
- board size 73.5 x 52 mm -> 58.4 x 52 mm
Changed lines of the file:
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@@
 <board>
 <plain>
-<wire x1="-0.0762" y1="8.6106" x2="73.3352" y2="8.5598" width="0" layer="20"/>
-<wire x1="73.3352" y1="8.5598" x2="73.259" y2="60.5792" width="0" layer="20"/>
-<wire x1="73.259" y1="60.5792" x2="-0.1524" y2="60.4522" width="0" layer="20"/>
+<wire x1="-0.0762" y1="8.6106" x2="58.2222" y2="8.4582" width="0" layer="20"/>
+<wire x1="58.2222" y1="8.4582" x2="58.146" y2="60.4776" width="0" layer="20"/>
+<wire x1="58.146" y1="60.4776" x2="-0.1524" y2="60.4522" width="0" layer="20"/>
 <wire x1="-0.1524" y1="60.4522" x2="-0.0762" y2="8.6106" width="0" layer="20"/>
-<hole x="1.778" y="58.4454" drill="3.175"/>
-<hole x="2.1844" y="10.8712" drill="3.175"/>
-<hole x="62.992" y="10.7696" drill="3.175"/>
-<hole x="63.119" y="58.5216" drill="3.175"/>
-<rectangle x1="0.6096" y1="58.0898" x2="0.8382" y2="58.2168" layer="16"/>
-<rectangle x1="57.9882" y1="18.5928" x2="70.9676" y2="35.6362" layer="16"/>
-<rectangle x1="58.0644" y1="36.6014" x2="71.0438" y2="53.6448" layer="16"/>
-<rectangle x1="59.055" y1="36.6014" x2="65.5574" y2="49.276" layer="45"/>
-<rectangle x1="59.055" y1="22.987" x2="65.5574" y2="35.6616" layer="45"/>
+<hole x="3.2512" y="57.277" drill="3.175"/>
+<hole x="3.0734" y="11.6586" drill="3.175"/>
+<hole x="54.0766" y="12.1666" drill="3.175"/>
+<hole x="54.7624" y="57.5564" drill="3.175"/>
 </plain>
 <attributes>
@@
 <elements>
 <element name="U$1" library="Spark" package="PHOTON" value="PHOTON_WITH_HEADERS" x="15.24" y="17.78"/>
-<element name="J2" library="SparkFun-Connectors" package="SCREWTERMINAL-3.5MM-2" value="" x="2.4638" y="43.8404" rot="R90">
-<attribute name="PROD_ID" value="CONN-08399" x="2.4638" y="43.8404" size="1.778" layer="27" rot="R90" display="off"/>
+<element name="J2" library="SparkFun-Connectors" package="SCREWTERMINAL-3.5MM-2" value="" x="5.7912" y="43.7388" rot="R90">
+<attribute name="PROD_ID" value="CONN-08399" x="5.7912" y="43.7388" size="1.778" layer="27" rot="R90" display="off"/>
 </element>
 <element name="R2" library="resistor" library_urn="urn:adsk.eagle:library:348" package="0207/10" package3d_urn="urn:adsk.eagle:package:25939/1" value="" x="10.4902" y="19.6596" rot="R90"/>
@@
 <contactref element="R1" pad="1"/>
 <contactref element="J2" pad="2"/>
-<wire x1="2.4638" y1="47.3404" x2="10.3378" y2="47.3404" width="1.5" layer="16"/>
+<wire x1="5.7912" y1="47.2388" x2="10.3378" y2="47.3404" width="1.5" layer="16"/>
 <wire x1="10.3378" y1="47.3404" x2="16.51" y2="47.3404" width="1.5" layer="16"/>
 <wire x1="16.51" y1="47.3404" x2="16.51" y2="47.498" width="0.6096" layer="16"/>
@@
 <contactref element="J2" pad="1"/>
 <contactref element="R2" pad="1"/>
-<wire x1="2.4638" y1="43.8404" x2="2.4638" y2="14.5796" width="1.5" layer="16"/>
-<wire x1="2.4638" y1="14.5796" x2="10.4902" y2="14.5796" width="1.5" layer="16"/>
+<wire x1="5.7912" y1="43.7388" x2="5.7912" y2="14.5796" width="1.5" layer="16"/>
+<wire x1="5.7912" y1="14.5796" x2="10.4902" y2="14.5796" width="1.5" layer="16"/>
 </signal>
 </signals>

Commit message: header swap
Parts:
- removed IC1: ACS750LCA-050, allegro:ACS75050
- added SV1: (no value), con-lstb:MA03-1
Connections:
- net N$1: now also SV1.3; no longer IC1.1
- net N$2: now also SV1.2; no longer IC1.2
- net N$3: now also SV1.1; no longer IC1.3
Routing:
- net N$1: track 18.8 -> 18.2 mm
Changed lines of the file:
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@@
 <element name="R2" library="resistor" library_urn="urn:adsk.eagle:library:348" package="0207/10" package3d_urn="urn:adsk.eagle:package:25939/1" value="" x="10.4902" y="19.6596" rot="R90"/>
 <element name="R1" library="resistor" library_urn="urn:adsk.eagle:library:348" package="0207/10" package3d_urn="urn:adsk.eagle:package:25939/1" value="" x="10.3378" y="33.1724" rot="R270"/>
-<element name="IC1" library="allegro" library_urn="urn:adsk.eagle:library:93" package="ACS75050" package3d_urn="urn:adsk.eagle:package:3457/1" value="ACS750LCA-050" x="62.2554" y="36.068" rot="R270">
-<attribute name="MF" value="ALLEGRO MICROSYSTEMS, INC." x="62.2554" y="36.068" size="1.778" layer="27" rot="R270" display="off"/>
-<attribute name="MPN" value="ACS750LCA-050" x="62.2554" y="36.068" size="1.778" layer="27" rot="R270" display="off"/>
-<attribute name="OC_FARNELL" value="1457176" x="62.2554" y="36.068" size="1.778" layer="27" rot="R270" display="off"/>
-<attribute name="OC_NEWARK" value="61H4464" x="62.2554" y="36.068" size="1.778" layer="27" rot="R270" display="off"/>
+<element name="SV1" library="con-lstb" library_urn="urn:adsk.eagle:library:162" package="MA03-1" package3d_urn="urn:adsk.eagle:package:8339/1" value="" x="41.1226" y="36.2458" rot="R90">
+<attribute name="MF" value="" x="41.1226" y="36.2458" size="1.778" layer="27" rot="R90" display="off"/>
+<attribute name="MPN" value="" x="41.1226" y="36.2458" size="1.778" layer="27" rot="R90" display="off"/>
+<attribute name="OC_FARNELL" value="unknown" x="41.1226" y="36.2458" size="1.778" layer="27" rot="R90" display="off"/>
+<attribute name="OC_NEWARK" value="unknown" x="41.1226" y="36.2458" size="1.778" layer="27" rot="R90" display="off"/>
 </element>
 </elements>
@@
 <contactref element="U$1" pad="24"/>
 <wire x1="34.29" y1="49.8856" x2="34.29" y2="50.038" width="0.6096" layer="16"/>
-<contactref element="IC1" pad="1"/>
 <wire x1="34.29" y1="50.038" x2="40.8554" y2="50.038" width="1.5" layer="16"/>
-<wire x1="40.8554" y1="50.038" x2="40.8554" y2="37.978" width="1.5" layer="16"/>
+<contactref element="SV1" pad="3"/>
+<wire x1="40.8554" y1="50.038" x2="40.8554" y2="38.7858" width="1.5" layer="16"/>
+<wire x1="40.8554" y1="38.7858" x2="41.1226" y2="38.7858" width="1.5" layer="16"/>
 </signal>
 <signal name="N$2">
 <contactref element="U$1" pad="21"/>
 <wire x1="34.4678" y1="42.5196" x2="34.544" y2="41.91" width="0.4064" layer="16"/>
-<contactref element="IC1" pad="2"/>
-<wire x1="40.8554" y1="36.068" x2="37.7444" y2="36.068" width="1.5" layer="16"/>
-<wire x1="37.7444" y1="36.068" x2="37.7444" y2="42.2656" width="1.5" layer="16"/>
+<wire x1="37.7444" y1="42.2656" x2="37.7444" y2="36.068" width="1.5" layer="16"/>
 <wire x1="37.7444" y1="42.2656" x2="34.29" y2="42.2656" width="1.5" layer="16"/>
 <wire x1="34.29" y1="42.2656" x2="34.29" y2="42.418" width="1.27" layer="16"/>
+<contactref element="SV1" pad="2"/>
+<wire x1="37.7444" y1="36.068" x2="41.1226" y2="36.068" width="1.5" layer="16"/>
+<wire x1="41.1226" y1="36.068" x2="41.1226" y2="36.2458" width="1.5" layer="16"/>
 <wire x1="34.29" y1="42.418" x2="34.4678" y2="42.5196" width="0" layer="19" extent="16-16"/>
 </signal>
@@
 <contactref element="U$1" pad="12"/>
 <wire x1="16.5608" y1="22.098" x2="16.51" y2="22.098" width="0.508" layer="16"/>
-<contactref element="IC1" pad="3"/>
-<wire x1="16.51" y1="22.098" x2="16.51" y2="14.9606" width="1.5" layer="16"/>
-<wire x1="40.8554" y1="14.9606" x2="40.8554" y2="34.158" width="1.5" layer="16"/>
-<wire x1="16.51" y1="14.9606" x2="40.8554" y2="14.9606" width="1.5" layer="16"/>
+<wire x1="16.51" y1="14.9606" x2="16.51" y2="22.098" width="1.5" layer="16"/>
+<contactref element="SV1" pad="1"/>
+<wire x1="41.1226" y1="33.7058" x2="41.1226" y2="14.9606" width="1.5" layer="16"/>
+<wire x1="41.1226" y1="14.9606" x2="16.51" y2="14.9606" width="1.5" layer="16"/>
 </signal>
 <signal name="VIN">
