File: hardware/ygl_energy_monitor.sch (EAGLE design)
At the start: 5 parts

Commit message: fixed package
Parts:
- removed U$2: (no value), LEM:HO_P_SP33
- added SV1: (no value), con-lstb:MA03-1
Connections:
- net N$1: now also SV1.1; no longer U$2.V_CC
- net N$2: now also SV1.2; no longer U$2.GND
- net N$3: now also SV1.3; no longer U$2.V_OUT
Changed lines of the file:
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@@
 </classes>
 <parts>
-<part name="U$2" library="LEM" deviceset="HO_P_SP33" device=""/>
 <part name="U$1" library="Spark" deviceset="PHOTON" device="_WITH_HEADERS"/>
 <part name="J2" library="SparkFun-Connectors" deviceset="CONN_02" device="3.5MM"/>
 <part name="R2" library="resistor" library_urn="urn:adsk.eagle:library:348" deviceset="R-US_" device="0207/10" package3d_urn="urn:adsk.eagle:package:25939/1"/>
 <part name="R1" library="resistor" library_urn="urn:adsk.eagle:library:348" deviceset="R-US_" device="0207/10" package3d_urn="urn:adsk.eagle:package:25939/1"/>
+<part name="SV1" library="con-lstb" library_urn="urn:adsk.eagle:library:162" deviceset="MA03-1" device="" package3d_urn="urn:adsk.eagle:package:8339/1"/>
 </parts>
 <sheets>
@@
 </plain>
 <instances>
-<instance part="U$2" gate="G$1" x="83.82" y="55.88"/>
 <instance part="U$1" gate="G$1" x="43.18" y="40.64"/>
 <instance part="J2" gate="G$1" x="-2.54" y="25.4"/>
 <instance part="R2" gate="G$1" x="10.16" y="38.1" rot="R90"/>
 <instance part="R1" gate="G$1" x="10.16" y="53.34" rot="R270"/>
+<instance part="SV1" gate="G$1" x="96.52" y="60.96" rot="R180"/>
 </instances>
 <busses>
@@
 <segment>
 <pinref part="U$1" gate="G$1" pin="3V3"/>
-<pinref part="U$2" gate="G$1" pin="V_CC"/>
 <wire x1="60.96" y1="68.58" x2="88.9" y2="68.58" width="0.1524" layer="91"/>
 <wire x1="88.9" y1="68.58" x2="88.9" y2="63.5" width="0.1524" layer="91"/>
+<pinref part="SV1" gate="G$1" pin="1"/>
 </segment>
 </net>
@@
 <wire x1="60.96" y1="53.34" x2="76.2" y2="53.34" width="0.1524" layer="91"/>
 <wire x1="76.2" y1="53.34" x2="76.2" y2="60.96" width="0.1524" layer="91"/>
-<pinref part="U$2" gate="G$1" pin="GND"/>
 <wire x1="76.2" y1="60.96" x2="88.9" y2="60.96" width="0.1524" layer="91"/>
+<pinref part="SV1" gate="G$1" pin="2"/>
 </segment>
 </net>
 <net name="N$3" class="0">
 <segment>
-<pinref part="U$2" gate="G$1" pin="V_OUT"/>
 <wire x1="88.9" y1="58.42" x2="78.74" y2="58.42" width="0.1524" layer="91"/>
 <wire x1="78.74" y1="58.42" x2="78.74" y2="48.26" width="0.1524" layer="91"/>
@@
 <wire x1="63.5" y1="7.62" x2="25.4" y2="7.62" width="0.1524" layer="91"/>
 <wire x1="25.4" y1="7.62" x2="25.4" y2="12.7" width="0.1524" layer="91"/>
+<pinref part="SV1" gate="G$1" pin="3"/>
 </segment>
 </net>

Commit message: embrace the braze!
Parts:
- removed SV1: (no value), con-lstb:MA03-1
- added IC1: ACS750LCA-050, allegro:ACS750LCA-050
Connections:
- net N$1: now also IC1.VCC; no longer SV1.1
- net N$2: now also IC1.GND; no longer SV1.2
- net N$3: now also IC1.VOUT; no longer SV1.3
Changed lines of the file:
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@@
 <part name="R2" library="resistor" library_urn="urn:adsk.eagle:library:348" deviceset="R-US_" device="0207/10" package3d_urn="urn:adsk.eagle:package:25939/1"/>
 <part name="R1" library="resistor" library_urn="urn:adsk.eagle:library:348" deviceset="R-US_" device="0207/10" package3d_urn="urn:adsk.eagle:package:25939/1"/>
-<part name="SV1" library="con-lstb" library_urn="urn:adsk.eagle:library:162" deviceset="MA03-1" device="" package3d_urn="urn:adsk.eagle:package:8339/1"/>
+<part name="IC1" library="allegro" library_urn="urn:adsk.eagle:library:93" deviceset="ACS750*CA-050" device="" package3d_urn="urn:adsk.eagle:package:3457/1" technology="L"/>
 </parts>
 <sheets>
@@
 <instance part="R2" gate="G$1" x="10.16" y="38.1" rot="R90"/>
 <instance part="R1" gate="G$1" x="10.16" y="53.34" rot="R270"/>
-<instance part="SV1" gate="G$1" x="96.52" y="60.96" rot="R180"/>
+<instance part="IC1" gate="G$1" x="93.98" y="45.72" rot="R180"/>
 </instances>
 <busses>
@@
 <segment>
 <pinref part="U$1" gate="G$1" pin="3V3"/>
-<wire x1="60.96" y1="68.58" x2="88.9" y2="68.58" width="0.1524" layer="91"/>
-<wire x1="88.9" y1="68.58" x2="88.9" y2="63.5" width="0.1524" layer="91"/>
-<pinref part="SV1" gate="G$1" pin="1"/>
+<wire x1="60.96" y1="68.58" x2="81.28" y2="68.58" width="0.1524" layer="91"/>
+<pinref part="IC1" gate="G$1" pin="VCC"/>
+<wire x1="83.82" y1="40.64" x2="81.28" y2="40.64" width="0.1524" layer="91"/>
+<wire x1="81.28" y1="40.64" x2="81.28" y2="68.58" width="0.1524" layer="91"/>
 </segment>
 </net>
@@
 <pinref part="U$1" gate="G$1" pin="GND@21"/>
 <wire x1="60.96" y1="53.34" x2="76.2" y2="53.34" width="0.1524" layer="91"/>
-<wire x1="76.2" y1="53.34" x2="76.2" y2="60.96" width="0.1524" layer="91"/>
-<wire x1="76.2" y1="60.96" x2="88.9" y2="60.96" width="0.1524" layer="91"/>
-<pinref part="SV1" gate="G$1" pin="2"/>
+<pinref part="IC1" gate="G$1" pin="GND"/>
+<wire x1="76.2" y1="53.34" x2="76.2" y2="50.8" width="0.1524" layer="91"/>
+<wire x1="76.2" y1="50.8" x2="83.82" y2="50.8" width="0.1524" layer="91"/>
 </segment>
 </net>
 <net name="N$3" class="0">
 <segment>
-<wire x1="88.9" y1="58.42" x2="78.74" y2="58.42" width="0.1524" layer="91"/>
-<wire x1="78.74" y1="58.42" x2="78.74" y2="48.26" width="0.1524" layer="91"/>
 <wire x1="78.74" y1="48.26" x2="63.5" y2="48.26" width="0.1524" layer="91"/>
 <wire x1="63.5" y1="48.26" x2="63.5" y2="7.62" width="0.1524" layer="91"/>
@@
 <wire x1="63.5" y1="7.62" x2="25.4" y2="7.62" width="0.1524" layer="91"/>
 <wire x1="25.4" y1="7.62" x2="25.4" y2="12.7" width="0.1524" layer="91"/>
-<pinref part="SV1" gate="G$1" pin="3"/>
+<pinref part="IC1" gate="G$1" pin="VOUT"/>
+<wire x1="78.74" y1="48.26" x2="78.74" y2="45.72" width="0.1524" layer="91"/>
+<wire x1="78.74" y1="45.72" x2="83.82" y2="45.72" width="0.1524" layer="91"/>
 </segment>
 </net>

Commit message: header swap
Parts:
- removed IC1: ACS750LCA-050, allegro:ACS750LCA-050
- added SV1: (no value), con-lstb:MA03-1
Connections:
- net N$1: now also SV1.3; no longer IC1.VCC
- net N$2: now also SV1.2; no longer IC1.GND
- net N$3: now also SV1.1; no longer IC1.VOUT
